File: boards/rev3-noserial.brd (EAGLE design)
At the start: 39.4 x 83.8 mm, 36 parts, among them IC1 AZ1117CR-3.3TRG1, U1 ESP32-S2-SOLO-2-N4

Commit message: Update the no-serial design for autoprogram.
This includes the same design block as the ESP32 WROOM-like modules, which means it should be possible to auto-program the boards without needing to solder in buttons.
Parts:
- added Q1, Q2: L8050QLT1G, Transistor:SOT95P237X112-3N
- added R1, R3: 10K, rcl:R0805
- added R4, R8: 0, rcl:R0805
- moved C1 10.2 mm to (30.5, 52.1)
Connections:
- new net !DTR: Q2.2, R1.1, UART.1
- new net !RTS: Q1.2, R3.1, UART.6
- new net N$10: Q1.3, R4.1
- new net N$11: Q2.3, R8.1
- new net N$5: Q1.1, R1.2
- new net N$6: Q2.1, R3.2
- net ESP_BOOT: now also R8.2; no longer UART.1
- net ESP_EN: now also R4.2; no longer UART.6
Routing:
- net GND: track 378.9 -> 322.8 mm
- net +5V: track 232.0 -> 196.6 mm, vias 2 -> 9
- net !RTS: track 0.00 -> 26.3 mm
- net ESP_BOOT: track 54.1 -> 29.6 mm
- net !DTR: track 0.00 -> 24.0 mm
- net N$11: track 0.00 -> 17.9 mm
- net ESP_EN: track 78.4 -> 66.5 mm, vias 1 -> 0
- net N$6: track 0.00 -> 9.30 mm
- net N$5: track 0.00 -> 6.27 mm
- net 3V3: track 78.9 -> 84.8 mm, vias 3 -> 4
- net N$10: track 0.00 -> 5.85 mm
- net ESP_TX: track 51.3 -> 55.8 mm, vias 0 -> 1
- net ESP_RX: track 47.2 -> 44.7 mm, vias 0 -> 1
- net NEOPIXEL_DATA: track 82.0 -> 83.8 mm
Other:
- board text added: "!RTS GND RXD TXD +3V !DTR"
- board text added: "Neopixel Acrylic Lamp rev. 3.1 - Licensed under MIT Copyright © 2023 Diego Elio Pettenò - defp.uk/espacrylic"
- board text removed: "!RST GND RXD TXD +3V !BOOT"
- board text removed: "Neopixel Acrylic Lamp rev. 3 - Licensed under MIT Copyright © 2023 Diego Elio Pettenò - defp.uk/espacrylic"
